File: HW/LPRS1_MAX1000_Shield_v1.0/LPRS1_MAX1000_Shield/LPRS1_MAX1000_Shield.kicad_pcb (KiCad board)
At the start: 2 copper layers, 130 x 90 mm, 198 parts, among them J1 2x6 2.54mm female, J10 1x16 2.54mm female, J11 1x16 2.54mm female, J2 1x14 2.54mm female, J3 1x14 2.54mm female, J4 1x3 2.54mm female, J5 1x3 2.54mm male, J6 3.5 mm stereo female, J7 1x2 2.54mm male, J8 3.5 mm stereo female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

Commit message: Update to new KiCAD version.
Other:
- net class Default removed
- net class Thick removed
- net class Thin removed
