File: HW/Ard_Nano_2_LPRS1_MAX1000_Shield/Ard_Nano_2_LPRS1_MAX1000_Shield.kicad_pcb (KiCad board)
At the start: 2 copper layers, 3 parts, among them J2 1x14 2.54mm female, J3 1x14 2.54mm female

Commit message: Done shield.
Connections:
- A1 pad 10: /D7 -> /D7__D2
- A1 pad 11: /D8 -> /D8__D1
- A1 pad 14: /D11 -> /D11__AIN0
- A1 pad 16: /D13 -> /D13__AIN3
- A1 pad 20: /A1 -> /A1__D10
- A1 pad 21: /A2 -> /A2__D9
- A1 pad 22: /A3 -> /A3__D8
- A1 pad 23: /A4 -> /A4__D7
- A1 pad 5: /D2 -> /D2__AIN2
- A1 pad 6: /D3 -> /D3__AIN1
- A1 pad 8: /D5 -> /D5__D4
- A1 pad 9: /D6 -> /D6__D3
- J2 pad 2: unconnected-(J2-Pin_2-Pad2) -> /A4__D7
- J2 pad 3: unconnected-(J2-Pin_3-Pad3) -> /A3__D8
- J2 pad 4: unconnected-(J2-Pin_4-Pad4) -> /A2__D9
- J2 pad 5: unconnected-(J2-Pin_5-Pad5) -> /A1__D10
- J3 pad 10: unconnected-(J3-Pin_10-Pad10) -> /D8__D1
- J3 pad 11: unconnected-(J3-Pin_11-Pad11) -> /D7__D2
- J3 pad 12: unconnected-(J3-Pin_12-Pad12) -> /D6__D3
- J3 pad 13: unconnected-(J3-Pin_13-Pad13) -> /D5__D4
- J3 pad 2: unconnected-(J3-Pin_2-Pad2) -> /D11__AIN0
- J3 pad 3: unconnected-(J3-Pin_3-Pad3) -> /D3__AIN1
- J3 pad 4: unconnected-(J3-Pin_4-Pad4) -> /D2__AIN2
- J3 pad 5: unconnected-(J3-Pin_5-Pad5) -> /D13__AIN3
Routing:
- net /D2__AIN2: track 0.00 -> 48.3 mm, vias 0 -> 2
- net /D3__AIN1: track 0.00 -> 43.2 mm, vias 0 -> 2
- net /D13__AIN3: track 0.00 -> 20.3 mm
- net /D11__AIN0: track 0.00 -> 20.3 mm, vias 0 -> 2
- net /D8__D1: track 0.00 -> 2.54 mm
- net /D7__D2: track 0.00 -> 2.54 mm
- net /D6__D3: track 0.00 -> 2.54 mm
- net /D5__D4: track 0.00 -> 2.54 mm
- net /A4__D7: track 0.00 -> 2.54 mm
- net /A3__D8: track 0.00 -> 2.54 mm
- net /A2__D9: track 0.00 -> 2.54 mm
- net /A1__D10: track 0.00 -> 2.54 mm
Other:
- board outline added: 53.3 x 25.4 mm

Commit message: Optimizing.
Parts:
- renumbered J2 to J1, J3 to J2
Connections:
- J2 pad 1: +2V5 -> unconnected-(J2-Pin_1-Pad1)

Commit message: This is correct way.
Parts:
- A1: moved to F.Cu
- moved A1 16.1 mm to (86.4, 81.3), turned to 90 degrees
Connections:
- A1 pad 29: GND -> unconnected-(A1-GND-Pad29)
- A1 pad 4: unconnected-(A1-GND-Pad4) -> GND
Routing:
- net /D2__AIN2: track 48.3 -> 0.00 mm, vias 2 -> 0
- net /D3__AIN1: track 43.2 -> 0.00 mm, vias 2 -> 0
- net /D13__AIN3: track 20.3 -> 0.00 mm
- net /D11__AIN0: track 20.3 -> 0.00 mm, vias 2 -> 0
- net /D10__D12: track 17.8 -> 0.00 mm
- net GND: track 45.7 -> 35.6 mm
- net /D9__D0: track 2.54 -> 0.00 mm
- net /D8__D1: track 2.54 -> 0.00 mm
- net /D7__D2: track 2.54 -> 0.00 mm
- net /D6__D3: track 2.54 -> 0.00 mm
- net /D5__D4: track 2.54 -> 0.00 mm
- net /D4__D5: track 2.54 -> 0.00 mm
- net /D12__AIN4: track 2.54 -> 0.00 mm
- net /A5__D6: track 2.54 -> 0.00 mm
- net /A4__D7: track 2.54 -> 0.00 mm
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
Commit message: Better.
Parts:
- moved A1 2.54 mm to (83.8, 81.3)
Routing:
- net GND: track 35.6 -> 38.1 mm
- net +5V: track 53.3 -> 55.9 mm
Other:
- board size 53.3 x 25.4 mm -> 50.8 x 25.4 mm
Changed lines of the file:
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@@
 	(footprint "Module:Arduino_Nano"
 		(layer "F.Cu")
-		(at 86.36 81.28 90)
+		(at 83.82 81.28 90)
 		(descr "Arduino Nano, http://www.mouser.com/pdfdocs/Gravitech_Arduino_Nano3_0.pdf")
 		(tags "Arduino Nano")
@@
 	(gr_line
 		(start 93.98 83.82)
-		(end 78.74 83.82)
+		(end 81.28 83.82)
 		(stroke
 			(width 0.05)
@@
 	)
 	(gr_line
-		(start 78.74 60.96)
+		(start 81.28 60.96)
 		(end 132.08 60.96)
 		(stroke
@@
 	)
 	(gr_line
-		(start 78.74 83.82)
-		(end 78.74 60.96)
+		(start 132.08 60.96)
+		(end 132.08 86.36)
+		(stroke
+			(width 0.05)
+			(type default)
+		)
+		(layer "Edge.Cuts")
+	)
+	(gr_line
+		(start 81.28 83.82)
+		(end 81.28 60.96)
 		(stroke
 			(width 0.05)
@@
 	)
 	(segment
-		(start 93.98 78.74)
-		(end 124.46 78.74)
+		(start 91.44 78.74)
+		(end 121.92 78.74)
 		(width 2)
 		(layer "F.Cu")
@@
 	)
 	(via
-		(at 93.98 78.74)
+		(at 91.44 78.74)
 		(size 2)
 		(drill 1)
@@
 	)
 	(via
-		(at 124.46 78.74)
+		(at 121.92 78.74)
 		(size 2)
 		(drill 1)
@@
 	)
 	(segment
-		(start 93.98 81.28)
-		(end 93.98 78.74)
+		(start 91.44 81.28)
+		(end 91.44 78.74)
 		(width 2)
 		(layer "B.Cu")
@@
 	)
 	(segment
-		(start 124.46 78.74)
-		(end 124.46 81.28)
+		(start 121.92 78.74)
+		(end 121.92 83.82)
 		(width 2)
 		(layer "B.Cu")
@@
 	(segment
 		(start 129.54 73.66)
-		(end 93.98 73.66)
+		(end 91.44 73.66)
 		(width 2)
 		(layer "F.Cu")
@@
 	)
 	(via
-		(at 93.98 73.66)
+		(at 91.44 73.66)
 		(size 2)
 		(drill 1)
@@
 	)
 	(segment
-		(start 93.98 73.66)
-		(end 93.98 66.04)
+		(start 91.44 73.66)
+		(end 91.44 66.04)
 		(width 2)
 		(layer "B.Cu")

Commit message: Done.
Connections:
- A1 pad 10: /D7__D2 -> /D7__D10
- A1 pad 11: /D8__D1 -> /D8__D11
- A1 pad 12: /D9__D0 -> /D9__D12
- A1 pad 13: /D10__D12 -> /D10__AIN1
- A1 pad 14: /D11__AIN0 -> /D11__AIN4
- A1 pad 15: /D12__AIN4 -> /D12__AIN0
- A1 pad 18: /D10__D12 -> unconnected-(A1-AREF-Pad18)
- A1 pad 19: /A0__D11 -> /A0__AIN2
- A1 pad 20: /A1__D10 -> /A1__D0
- A1 pad 21: /A2__D9 -> /A2__D1
- A1 pad 22: /A3__D8 -> /A3__D2
- A1 pad 23: /A4__D7 -> /A4__D3
- A1 pad 24: /A5__D6 -> /A5__D4
- A1 pad 5: /D2__AIN2 -> /D2__D5
- A1 pad 6: /D3__AIN1 -> /D3__D6
- A1 pad 7: /D4__D5 -> /D4__D7
- A1 pad 8: /D5__D4 -> /D5__D8
- A1 pad 9: /D6__D3 -> /D6__D9
- J1 pad 1: /A5__D6 -> /D3__D6
- J1 pad 2: /A4__D7 -> /D4__D7
- J1 pad 3: /A3__D8 -> /D5__D8
- J1 pad 4: /A2__D9 -> /D6__D9
- J1 pad 5: /A1__D10 -> /D7__D10
- J1 pad 6: /A0__D11 -> /D8__D11
- J1 pad 7: /D10__D12 -> /D9__D12
- J2 pad 10: /D8__D1 -> /A2__D1
- J2 pad 11: /D7__D2 -> /A3__D2
- J2 pad 12: /D6__D3 -> /A4__D3
- J2 pad 13: /D5__D4 -> /A5__D4
- J2 pad 14: /D4__D5 -> /D2__D5
- J2 pad 2: /D11__AIN0 -> /D12__AIN0
- J2 pad 3: /D3__AIN1 -> /D10__AIN1
- J2 pad 4: /D2__AIN2 -> /A0__AIN2
- J2 pad 6: /D12__AIN4 -> /D11__AIN4
- J2 pad 9: /D9__D0 -> /A1__D0
Routing:
- net /D10__AIN1: track 0.00 -> 27.9 mm, vias 0 -> 2
- net /D12__AIN0: track 0.00 -> 25.4 mm, vias 0 -> 2
- net /A0__AIN2: track 0.00 -> 17.8 mm, vias 0 -> 2
- net /D2__D5: track 0.00 -> 15.2 mm
- net /D11__AIN4: track 0.00 -> 12.7 mm
- net /D13__AIN3: track 0.00 -> 2.54 mm
- net /A5__D4: track 0.00 -> 2.54 mm
- net /A4__D3: track 0.00 -> 2.54 mm
- net /A3__D2: track 0.00 -> 2.54 mm
- net /A2__D1: track 0.00 -> 2.54 mm
- net /A1__D0: track 0.00 -> 2.54 mm
- net /D9__D12: track 0.00 -> 2.54 mm
- net /D8__D11: track 0.00 -> 2.54 mm
- net /D7__D10: track 0.00 -> 2.54 mm
- net /D6__D9: track 0.00 -> 2.54 mm
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
Commit message: 3V3
Connections:
- A1 pad 17: unconnected-(A1-3V3-Pad17) -> +3V3
- J1 pad 12: unconnected-(J1-Pin_12-Pad12) -> +3V3
Routing:
- net +3V3: track 0.00 -> 25.4 mm, vias 0 -> 2
- net /D10__AIN1: track 27.9 -> 12.7 mm, vias 2 -> 0
- net /D11__AIN4: track 12.7 -> 25.4 mm, vias 0 -> 2
- net GND: track 38.1 -> 48.3 mm
- net /D12__AIN0: track 25.4 -> 20.3 mm
- net +5V: track 55.9 -> 61.0 mm
Other:
- board size 50.8 x 25.4 mm -> 50.8 x 30.5 mm

Commit message: New way.
Connections:
- A1 pad 13: /D10__AIN1 -> /D10__AIN4
- A1 pad 14: /D11__AIN4 -> /D11__AIN0
- A1 pad 15: /D12__AIN0 -> /D12__AIN1
- J2 pad 2: /D12__AIN0 -> /D11__AIN0
- J2 pad 3: /D10__AIN1 -> /D12__AIN1
- J2 pad 6: /D11__AIN4 -> /D10__AIN4
Routing:
- net /D11__AIN4: track 25.4 -> 0.00 mm, vias 2 -> 0
- net /D12__AIN1: track 0.00 -> 20.3 mm, vias 0 -> 2
- net /D12__AIN0: track 20.3 -> 0.00 mm, vias 2 -> 0
- net /D11__AIN0: track 0.00 -> 17.8 mm
- net /D10__AIN4: track 0.00 -> 12.7 mm
- net /D10__AIN1: track 12.7 -> 0.00 mm
Changed lines of the file:
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@@
 	(net 29 "/D7__D10")
 	(net 30 "/A2__D1")
-	(net 31 "/D11__AIN4")
+	(net 31 "/D11__AIN0")
 	(net 32 "/D4__D7")
 	(net 33 "/D3__D6")
 	(net 34 "/D6__D9")
 	(net 35 "/A5__D4")
-	(net 36 "/D12__AIN0")
-	(net 37 "/D10__AIN1")
+	(net 36 "/D12__AIN1")
+	(net 37 "/D10__AIN4")
 	(footprint "Connector_PinSocket_2.54mm:PinSocket_1x14_P2.54mm_Vertical"
 		(layer "F.Cu")
@@
 			)
 			(remove_unused_layers no)
-			(net 36 "/D12__AIN0")
+			(net 31 "/D11__AIN0")
 			(pinfunction "Pin_2")
 			(pintype "passive")
@@
 			)
 			(remove_unused_layers no)
-			(net 37 "/D10__AIN1")
+			(net 36 "/D12__AIN1")
 			(pinfunction "Pin_3")
 			(pintype "passive")
@@
 			)
 			(remove_unused_layers no)
-			(net 31 "/D11__AIN4")
+			(net 37 "/D10__AIN4")
 			(pinfunction "Pin_6")
 			(pintype "passive")
@@
 			)
 			(remove_unused_layers no)
-			(net 37 "/D10__AIN1")
+			(net 37 "/D10__AIN4")
 			(pinfunction "D10")
 			(pintype "bidirectional")
@@
 			)
 			(remove_unused_layers no)
-			(net 31 "/D11__AIN4")
+			(net 31 "/D11__AIN0")
 			(pinfunction "D11")
 			(pintype "bidirectional")
@@
 			)
 			(remove_unused_layers no)
-			(net 36 "/D12__AIN0")
+			(net 36 "/D12__AIN1")
 			(pinfunction "D12")
 			(pintype "bidirectional")
@@
 	)
 	(segment
-		(start 116.84 86.36)
-		(end 127 86.36)
-		(width 2)
-		(layer "F.Cu")
-		(net 31)
-	)
-	(via
-		(at 127 86.36)
-		(size 2)
-		(drill 1)
-		(layers "F.Cu" "B.Cu")
-		(net 31)
-	)
-	(via
-		(at 116.84 86.36)
-		(size 2)
-		(drill 1)
-		(layers "F.Cu" "B.Cu")
-		(net 31)
-	)
-	(segment
-		(start 127 81.28)
-		(end 127 66.04)
+		(start 127 63.5)
+		(end 127 81.28)
 		(width 2)
 		(layer "B.Cu")

Commit message: Another swap.
Connections:
- A1 pad 13: /D10__AIN4 -> /D10__AIN2
- A1 pad 19: /A0__AIN2 -> /A0__AIN4
- J2 pad 4: /A0__AIN2 -> /D10__AIN2
- J2 pad 6: /D10__AIN4 -> /A0__AIN4
Routing:
- net /D10__AIN2: track 0.00 -> 25.4 mm, vias 0 -> 2
- net /A0__AIN2: track 17.8 -> 0.00 mm, vias 2 -> 0
- net /D10__AIN4: track 12.7 -> 0.00 mm
Changed lines of the file:
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@@
 	(net 24 "/D9__D12")
 	(net 25 "/A1__D0")
-	(net 26 "/A0__AIN2")
+	(net 26 "/A0__AIN4")
 	(net 27 "/D2__D5")
 	(net 28 "/A3__D2")
@@
 	(net 35 "/A5__D4")
 	(net 36 "/D12__AIN1")
-	(net 37 "/D10__AIN4")
+	(net 37 "/D10__AIN2")
 	(footprint "Connector_PinSocket_2.54mm:PinSocket_1x14_P2.54mm_Vertical"
 		(layer "F.Cu")
@@
 			)
 			(remove_unused_layers no)
-			(net 26 "/A0__AIN2")
+			(net 37 "/D10__AIN2")
 			(pinfunction "Pin_4")
 			(pintype "passive")
@@
 			)
 			(remove_unused_layers no)
-			(net 37 "/D10__AIN4")
+			(net 26 "/A0__AIN4")
 			(pinfunction "Pin_6")
 			(pintype "passive")
@@
 			)
 			(remove_unused_layers no)
-			(net 37 "/D10__AIN4")
+			(net 37 "/D10__AIN2")
 			(pinfunction "D10")
 			(pintype "bidirectional")
@@
 			)
 			(remove_unused_layers no)
-			(net 26 "/A0__AIN2")
+			(net 26 "/A0__AIN4")
 			(pinfunction "A0")
 			(pintype "bidirectional")
@@
 	)
 	(gr_line
-		(start 116.84 64.77)
+		(start 114.3 64.77)
 		(end 116.84 64.77)
 		(stroke
@@
 	)
 	(segment
-		(start 111.76 68.58)
-		(end 121.92 68.58)
-		(width 2)
-		(layer "F.Cu")
-		(net 26)
-	)
-	(via
-		(at 111.76 68.58)
-		(size 2)
-		(drill 1)
-		(layers "F.Cu" "B.Cu")
-		(net 26)
-	)
-	(via
-		(at 121.92 68.58)
-		(size 2)
-		(drill 1)
-		(layers "F.Cu" "B.Cu")
-		(net 26)
-	)
-	(segment
-		(start 111.76 66.04)
-		(end 111.76 68.58)
-		(width 2)
-		(layer "B.Cu")
-		(net 26)
-	)
-	(segment
-		(start 121.92 68.58)
-		(end 121.92 63.5)
-		(width 2)
-		(layer "B.Cu")
-		(net 26)
-	)
-	(segment
 		(start 96.52 63.5)
 		(end 93.98 63.5)
@@
 	)
 	(segment
+		(start 121.92 68.58)
+		(end 114.3 68.58)
+		(width 2)
+		(layer "F.Cu")
+		(net 37)
+	)
+	(via
+		(at 114.3 68.58)
+		(size 2)
+		(drill 1)
+		(layers "F.Cu" "B.Cu")
+		(net 37)
+	)
+	(via
+		(at 121.92 68.58)
+		(size 2)
+		(drill 1)
+		(layers "F.Cu" "B.Cu")
+		(net 37)
+	)
+	(segment
 		(start 114.3 81.28)
 		(end 114.3 73.66)
@@
 		(width 2)
 		(layer "B.Cu")
+		(net 37)
+	)
+	(segment
+		(start 121.92 68.58)
+		(end 121.92 63.5)
+		(width 2)
+		(layer "B.Cu")
