File: HW/Ard_Nano_2_LPRS1_MAX1000_Shield/Ard_Nano_2_LPRS1_MAX1000_Shield.kicad_pcb (KiCad board)
At the start: 2 copper layers, 50.8 x 30.5 mm, 3 parts, among them J1 1x14 2.54mm female, J2 1x14 2.54mm female

Commit message: v0.3
Connections:
- A1 pad 13: /D10__AIN2 -> /D10__AIN0
- A1 pad 14: /D11__AIN0 -> /D11__AIN4
- A1 pad 15: /D12__AIN1 -> /D12__AIN3
- A1 pad 16: /D13__AIN3 -> unconnected-(A1-D13-Pad16)
- A1 pad 17: +3V3 -> unconnected-(A1-3V3-Pad17)
- A1 pad 19: /A0__AIN4 -> /A0__AIN2
- J1 pad 12: +3V3 -> +5V
- J2 pad 2: /D11__AIN0 -> /D10__AIN0
- J2 pad 3: /D12__AIN1 -> unconnected-(J2-Pin_3-Pad3)
- J2 pad 4: /D10__AIN2 -> /A0__AIN2
- J2 pad 5: /D13__AIN3 -> /D12__AIN3
- J2 pad 6: /A0__AIN4 -> /D11__AIN4
Routing:
- net /D10__AIN0: track 0.00 -> 30.5 mm, vias 0 -> 2
- net /D10__AIN2: track 25.4 -> 0.00 mm, vias 2 -> 0
- net +3V3: track 25.4 -> 0.00 mm, vias 2 -> 0
- net /A0__AIN2: track 0.00 -> 22.9 mm, vias 0 -> 2
- net /D12__AIN1: track 20.3 -> 0.00 mm, vias 2 -> 0
- net /D11__AIN0: track 17.8 -> 0.00 mm
- net /D12__AIN3: track 0.00 -> 12.7 mm
- net /D11__AIN4: track 0.00 -> 12.7 mm
- net GND: track 48.3 -> 38.1 mm
- net +5V: track 61.0 -> 68.6 mm, vias 2 -> 4
- net /D13__AIN3: track 2.54 -> 0.00 mm
