File: HW/Ard_Nano_2_LPRS1_MAX1000_Shield/Ard_Nano_2_LPRS1_MAX1000_Shield.kicad_sch (KiCad schematic)
At the start: 3 parts, among them J2 1x14 2.54mm female, J3 1x14 2.54mm female

Commit message: Done shield.
Connections:
- net A1 is gone; now on net A1__D10: A1.20 (A1)
- net A2 is gone; now on net A2__D9: A1.21 (A2)
- net A3 is gone; now on net A3__D8: A1.22 (A3)
- net A4 is gone; now on net A4__D7: A1.23 (A4)
- net D11: no longer A1.14 (D11)
- net D13: no longer A1.16 (D13)
- net D2: no longer A1.5 (D2)
- net D3: no longer A1.6 (D3)
- net D5: no longer A1.8 (D5)
- net D6: no longer A1.9 (D6)
- net D7: no longer A1.10 (D7)
- net D8: no longer A1.11 (D8)
- net D8__D1: now reaches J3.10 (Pin_10)
- net D8__D1: now also A1.11 (D8)
- net D7__D2: now reaches J3.11 (Pin_11)
- net D7__D2: now also A1.10 (D7)
- net D6__D3: now reaches J3.12 (Pin_12)
- net D6__D3: now also A1.9 (D6)
- net D5__D4: now reaches J3.13 (Pin_13)
- net D5__D4: now also A1.8 (D5)
- net D11__AIN0: now reaches J3.2 (Pin_2)
- net D11__AIN0: now also A1.14 (D11)
- net D3__AIN1: now reaches J3.3 (Pin_3)
- net D3__AIN1: now also A1.6 (D3)
- net D2__AIN2: now reaches J3.4 (Pin_4)
- net D2__AIN2: now also A1.5 (D2)
- net D13__AIN3: now reaches J3.5 (Pin_5)
- net D13__AIN3: now also A1.16 (D13)
- net A4__D7: now reaches J2.2 (Pin_2)
- net A3__D8: now reaches J2.3 (Pin_3)
- net A2__D9: now reaches J2.4 (Pin_4)
- net A1__D10: now reaches J2.5 (Pin_5)

Commit message: Optimizing.
Parts:
- renumbered J2 to J1, J3 to J2
Connections:
- net +2V5: no longer names the net of J2.1 (Pin_1)
- no-connect marks 2 -> 15
Other:
- note added: "Pull out pin from connector for every you do not use A1: 1 2 3 4 17 18 25 26 28 30 J1: 8 9 10 12 13 J2: 1 7 8"
- note removed: "AREF"
Changed lines of the file:
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@@
 	(paper "A4")
 	(no_connect
+		(at 104.14 43.18)
+	)
+	(no_connect
+		(at 248.92 45.72)
+	)
+	(no_connect
+		(at 129.54 43.18)
+	)
+	(no_connect
+		(at 104.14 45.72)
+	)
+	(no_connect
 		(at 238.76 119.38)
+	)
+	(no_connect
+		(at 236.22 119.38)
+	)
+	(no_connect
+		(at 233.68 45.72)
+	)
+	(no_connect
+		(at 243.84 119.38)
+	)
+	(no_connect
+		(at 114.3 33.02)
+	)
+	(no_connect
+		(at 233.68 119.38)
+	)
+	(no_connect
+		(at 116.84 83.82)
+	)
+	(no_connect
+		(at 129.54 45.72)
 	)
 	(no_connect
 		(at 246.38 119.38)
 	)
+	(no_connect
+		(at 119.38 33.02)
+	)
+	(no_connect
+		(at 231.14 45.72)
+	)
 	(wire
 		(pts
@@
 	(wire
 		(pts
-			(xy 269.24 33.02) (xy 269.24 45.72)
-		)
-		(stroke
-			(width 0)
-			(type default)
-		)
-	)
-	(wire
-		(pts
 			(xy 91.44 63.5) (xy 104.14 63.5)
 		)
@@
 	(wire
 		(pts
-			(xy 248.92 33.02) (xy 248.92 45.72)
-		)
-		(stroke
-			(width 0)
-			(type default)
-		)
-	)
-	(wire
-		(pts
 			(xy 226.06 132.08) (xy 226.06 119.38)
 		)
@@
 		(pts
 			(xy 223.52 132.08) (xy 223.52 119.38)
-		)
-		(stroke
-			(width 0)
-			(type default)
-		)
-	)
-	(wire
-		(pts
-			(xy 257.81 33.02) (xy 248.92 33.02)
 		)
 		(stroke
@@
 		)
 	)
-	(text "AREF"
+	(text "Pull out pin from connector for every you do not use\nA1: 1 2 3 4 17 18 25 26 28 30\nJ1: 8 9 10 12 13\nJ2: 1 7 8"
 		(exclude_from_sim no)
-		(at 251.46 35.56 0)
-		(effects
-			(font
-				(size 1.27 1.27)
-			)
-			(justify left bottom)
+		(at 131.064 113.538 0)
+		(effects
+			(font
+				(size 1.27 1.27)
+			)
+			(justify left)
 		)
 	)
@@
 			)
 			(justify left bottom)
-		)
-	)
-	(label "D3__AIN0"
-		(at 269.24 33.02 270)
-		(effects
-			(font
-				(size 1.27 1.27)
-			)
-			(justify right bottom)
 		)
 	)
@@
 		(dnp no)
 		(fields_autoplaced yes)
-		(property "Reference" "#PWR3"
+		(property "Reference" "#PWR1"
 			(at 119.38 95.25 0)
 			(effects
@@
 			(project "Ard_Nano_2_LPRS1_MAX1000_Shield"
 				(path "/f032f0f5-bc12-4ceb-9247-9ea9649022af"
-					(reference "#PWR3")
+					(reference "#PWR1")
 					(unit 1)
 				)
@@
 		(on_board yes)
 		(dnp no)
-		(property "Reference" "#PWR4"
+		(property "Reference" "#PWR3"
 			(at 241.3 128.27 0)
 			(effects
@@
 			(project "Ard_Nano_2_LPRS1_MAX1000_Shield"
 				(path "/f032f0f5-bc12-4ceb-9247-9ea9649022af"
-					(reference "#PWR4")
+					(reference "#PWR3")
 					(unit 1)
 				)
@@
 		(on_board yes)
 		(dnp no)
-		(property "Reference" "J3"
+		(property "Reference" "J2"
 			(at 232.3084 53.975 90)
 			(effects
@@
 			(project "Ard_Nano_2_LPRS1_MAX1000_Shield"
 				(path "/f032f0f5-bc12-4ceb-9247-9ea9649022af"
-					(reference "J3")
+					(reference "J2")
 					(unit 1)
 				)
@@
 		(on_board yes)
 		(dnp no)
-		(property "Reference" "#PWR7"
+		(property "Reference" "#PWR4"
 			(at 248.92 118.11 0)
 			(effects
@@
 			(project "Ard_Nano_2_LPRS1_MAX1000_Shield"
 				(path "/f032f0f5-bc12-4ceb-9247-9ea9649022af"
-					(reference "#PWR7")
+					(reference "#PWR4")
 					(unit 1)
 				)
@@
 		(on_board yes)
 		(dnp no)
-		(property "Reference" "#PWR1"
+		(property "Reference" "#PWR2"
 			(at 121.92 34.29 0)
 			(effects
@@
 			(project "Ard_Nano_2_LPRS1_MAX1000_Shield"
 				(path "/f032f0f5-bc12-4ceb-9247-9ea9649022af"
-					(reference "#PWR1")
-					(unit 1)
-				)
-			)
-		)
-	)
-	(symbol
-		(lib_id "LPRS1_MAX1000_Shield-rescue:+2V5-power")
-		(at 257.81 33.02 0)
-		(unit 1)
-		(exclude_from_sim no)
-		(in_bom yes)
-		(on_board yes)
-		(dnp no)
-		(property "Reference" "#PWR8"
-			(at 257.81 36.83 0)
-			(effects
-				(font
-					(size 1.27 1.27)
-				)
-				(hide yes)
-			)
-		)
-		(property "Value" "+2V5"
-			(at 258.191 28.6258 0)
-			(effects
-				(font
-					(size 1.27 1.27)
-				)
-			)
-		)
-		(property "Footprint" ""
-			(at 257.81 33.02 0)
-			(effects
-				(font
-					(size 1.27 1.27)
-				)
-				(hide yes)
-			)
-		)
-		(property "Datasheet" ""
-			(at 257.81 33.02 0)
-			(effects
-				(font
-					(size 1.27 1.27)
-				)
-				(hide yes)
-			)
-		)
-		(property "Description" ""
-			(at 257.81 33.02 0)
-			(effects
-				(font
-					(size 1.27 1.27)
-				)
-				(hide yes)
-			)
-		)
-		(pin "1"
-		)
-		(instances
-			(project "Ard_Nano_2_LPRS1_MAX1000_Shield"
-				(path "/f032f0f5-bc12-4ceb-9247-9ea9649022af"
-					(reference "#PWR8")
+					(reference "#PWR2")
 					(unit 1)
 				)
@@
 		(on_board yes)
 		(dnp no)
-		(property "Reference" "J2"
+		(property "Reference" "J1"
 			(at 226.06 106.68 90)
 			(effects
@@
 			(project "Ard_Nano_2_LPRS1_MAX1000_Shield"
 				(path "/f032f0f5-bc12-4ceb-9247-9ea9649022af"
-					(reference "J2")
+					(reference "J1")
 					(unit 1)
 				)

Commit message: This is correct way.
Connections:
- net GND: now also A1.4 (GND); no longer A1.29 (GND)
- no-connect marks 15 -> 14
Changed lines of the file:
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@@
-	)
-	(no_connect
-		(at 116.84 83.82)
 	)
 	(no_connect
@@
 	(wire
 		(pts
-			(xy 119.38 83.82) (xy 119.38 88.9)
+			(xy 116.84 83.82) (xy 116.84 88.9)
 		)
 		(stroke
@@
 		(lib_name "GND_1")
 		(lib_id "power:GND")
-		(at 119.38 88.9 0)
+		(at 116.84 88.9 0)
 		(unit 1)
 		(exclude_from_sim no)
@@
 		(fields_autoplaced yes)
 		(property "Reference" "#PWR1"
-			(at 119.38 95.25 0)
+			(at 116.84 95.25 0)
 			(effects
 				(font
@@
 		)
 		(property "Value" "GND"
-			(at 119.3801 92.71 90)
+			(at 116.8401 92.71 90)
 			(effects
 				(font
@@
 		)
 		(property "Footprint" ""
-			(at 119.38 88.9 0)
+			(at 116.84 88.9 0)
 			(effects
 				(font
@@
 		)
 		(property "Datasheet" ""
-			(at 119.38 88.9 0)
+			(at 116.84 88.9 0)
 			(effects
 				(font
@@
 		)
 		(property "Description" "Power symbol creates a global label with name \"GND\" , ground"
-			(at 119.38 88.9 0)
+			(at 116.84 88.9 0)
 			(effects
 				(font

Commit message: Better.
Connections:
- net D10__D12: no longer A1.18 (AREF)
Other:
- note removed: "Pull out pin from female connector AREF"
Changed lines of the file:
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@@
-	(wire
-		(pts
-			(xy 142.24 53.34) (xy 129.54 53.34)
-		)
-		(stroke
-			(width 0)
-			(type default)
-		)
-	)
 	(wire
 		(pts
@@
 			(width 0)
 			(type default)
-		)
-	)
-	(text "Pull out pin from female connector AREF"
-		(exclude_from_sim no)
-		(at 165.608 53.086 0)
-		(effects
-			(font
-				(size 1.27 1.27)
-			)
 		)
 	)
@@
 		)
 	)
-	(label "D10__D12"
-		(at 142.24 53.34 180)
-		(effects
-			(font
-				(size 1.27 1.27)
-			)
-			(justify right bottom)
-		)
-	)

Commit message: Done.
Connections:
- net A0__D11 renamed A0__AIN2
- net A0__AIN2: now also J2.4 (Pin_4); no longer J1.6 (Pin_6)
- net A1__D10 renamed A1__D0
- net A1__D0: now also J2.9 (Pin_9); no longer J1.5 (Pin_5)
- net A2__D9 renamed A2__D1
- net A2__D1: now also J2.10 (Pin_10); no longer J1.4 (Pin_4)
- net A3__D8 renamed A3__D2
- net A3__D2: now also J2.11 (Pin_11); no longer J1.3 (Pin_3)
- net A4__D7 renamed A4__D3
- net A4__D3: now also J2.12 (Pin_12); no longer J1.2 (Pin_2)
- net A5__D6 renamed A5__D4
- net A5__D4: now also J2.13 (Pin_13); no longer J1.1 (Pin_1)
- net D10__D12 renamed D10__AIN1
- net D10__AIN1: now also J2.3 (Pin_3); no longer J1.7 (Pin_7)
- net D11__AIN0 renamed D11__AIN4
- net D11__AIN4: now also J2.6 (Pin_6); no longer J2.2 (Pin_2)
- net D12__AIN4 renamed D12__AIN0
- net D12__AIN0: now also J2.2 (Pin_2); no longer J2.6 (Pin_6)
- net D2__AIN2 renamed D2__D5
- net D2__D5: now also J2.14 (Pin_14); no longer J2.4 (Pin_4)
- net D3__AIN1 renamed D3__D6
- net D3__D6: now also J1.1 (Pin_1); no longer J2.3 (Pin_3)
- net D4__D5 renamed D4__D7
- net D4__D7: now also J1.2 (Pin_2); no longer J2.14 (Pin_14)
- net D5__D4 renamed D5__D8
- net D5__D8: now also J1.3 (Pin_3); no longer J2.13 (Pin_13)
- net D6__D3 renamed D6__D9
- net D6__D9: now also J1.4 (Pin_4); no longer J2.12 (Pin_12)
- net D7__D2 renamed D7__D10
- net D7__D10: now also J1.5 (Pin_5); no longer J2.11 (Pin_11)
- net D8__D1 renamed D8__D11
- net D8__D11: now also J1.6 (Pin_6); no longer J2.10 (Pin_10)
- net D9__D0 renamed D9__D12
- net D9__D12: now also J1.7 (Pin_7); no longer J2.9 (Pin_9)
- no-connect marks 14 -> 15
Other:
- note added: "Pull out pin from connector for every you do not use A1: 1 2 3 17 18 25 26 28 29 30 J1: 8 9 10 12 13 J2: 1 7 8"
- note removed: "Pull out pin from connector for every you do not use A1: 1 2 3 4 17 18 25 26 28 30 J1: 8 9 10 12 13 J2: 1 7 8"

Commit message: 3V3
Connections:
- net +3V3: now reaches A1.17 (3V3)
- net +3V3: now also J1.12 (Pin_12)
- no-connect marks 15 -> 13
Changed lines of the file:
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@@
-	)
-	(no_connect
-		(at 243.84 119.38)
 	)
 	(no_connect
@@
 	)
 	(no_connect
-		(at 119.38 33.02)
-	)
-	(no_connect
 		(at 231.14 45.72)
 	)
 	(wire
 		(pts
+			(xy 119.38 26.67) (xy 119.38 33.02)
+		)
+		(stroke
+			(width 0)
+			(type default)
+		)
+	)
+	(wire
+		(pts
 			(xy 91.44 66.04) (xy 104.14 66.04)
 		)
@@
 		(pts
 			(xy 142.24 60.96) (xy 129.54 60.96)
+		)
+		(stroke
+			(width 0)
+			(type default)
+		)
+	)
+	(wire
+		(pts
+			(xy 243.84 125.73) (xy 243.84 119.38)
 		)
 		(stroke
@@
 			)
 			(justify left bottom)
+		)
+	)
+	(symbol
+		(lib_id "LPRS1_MAX1000_Shield-rescue:+3V3-power")
+		(at 243.84 125.73 180)
+		(unit 1)
+		(exclude_from_sim no)
+		(in_bom yes)
+		(on_board yes)
+		(dnp no)
+		(property "Reference" "#PWR5"
+			(at 243.84 121.92 0)
+			(effects
+				(font
+					(size 1.27 1.27)
+				)
+				(hide yes)
+			)
+		)
+		(property "Value" "+3V3"
+			(at 243.459 130.1242 0)
+			(effects
+				(font
+					(size 1.27 1.27)
+				)
+			)
+		)
+		(property "Footprint" ""
+			(at 243.84 125.73 0)
+			(effects
+				(font
+					(size 1.27 1.27)
+				)
+				(hide yes)
+			)
+		)
+		(property "Datasheet" ""
+			(at 243.84 125.73 0)
+			(effects
+				(font
+					(size 1.27 1.27)
+				)
+				(hide yes)
+			)
+		)
+		(property "Description" ""
+			(at 243.84 125.73 0)
+			(effects
+				(font
+					(size 1.27 1.27)
+				)
+				(hide yes)
+			)
+		)
+		(pin "1"
+		)
+		(instances
+			(project "Ard_Nano_2_LPRS1_MAX1000_Shield"
+				(path "/f032f0f5-bc12-4ceb-9247-9ea9649022af"
+					(reference "#PWR5")
+					(unit 1)
+				)
+			)
 		)
 	)
@@
 					(unit 1)
 				)
+			)
+		)
+	)
+	(symbol
+		(lib_id "LPRS1_MAX1000_Shield-rescue:+3V3-power")
+		(at 119.38 26.67 0)
+		(unit 1)
+		(exclude_from_sim no)
+		(in_bom yes)
+		(on_board yes)
+		(dnp no)
+		(property "Reference" "#PWR6"
+			(at 119.38 30.48 0)
+			(effects
+				(font
+					(size 1.27 1.27)
+				)
+				(hide yes)
+			)
+		)
+		(property "Value" "+3V3"
+			(at 119.761 22.2758 0)
+			(effects
+				(font
+					(size 1.27 1.27)
+				)
+			)
+		)
+		(property "Footprint" ""
+			(at 119.38 26.67 0)
+			(effects
+				(font
+					(size 1.27 1.27)
+				)
+				(hide yes)
+			)
+		)
+		(property "Datasheet" ""
+			(at 119.38 26.67 0)
+			(effects
+				(font
+					(size 1.27 1.27)
+				)
+				(hide yes)
+			)
+		)
+		(property "Description" ""
+			(at 119.38 26.67 0)
+			(effects
+				(font
+					(size 1.27 1.27)
+				)
+				(hide yes)
+			)
+		)
+		(pin "1"
+		)
+		(instances
+			(project "Ard_Nano_2_LPRS1_MAX1000_Shield"
+				(path "/f032f0f5-bc12-4ceb-9247-9ea9649022af"
+					(reference "#PWR6")
+					(unit 1)
+				)

Commit message: New way.
Connections:
- net D10__AIN1 renamed D10__AIN4
- net D10__AIN4: now also J2.6 (Pin_6); no longer J2.3 (Pin_3)
- net D11__AIN4 renamed D11__AIN0
- net D11__AIN0: now also J2.2 (Pin_2); no longer J2.6 (Pin_6)
- net D12__AIN0 renamed D12__AIN1
- net D12__AIN1: now also J2.3 (Pin_3); no longer J2.2 (Pin_2)
Changed lines of the file:
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@@
 		)
 	)
-	(label "D11__AIN4"
+	(label "D11__AIN0"
 		(at 91.44 71.12 0)
 		(effects
@@
 		)
 	)
-	(label "D10__AIN1"
+	(label "D10__AIN4"
 		(at 91.44 68.58 0)
 		(effects
@@
 		)
 	)
-	(label "D12__AIN0"
+	(label "D12__AIN1"
 		(at 91.44 73.66 0)
 		(effects
@@
 		)
 	)
-	(label "D10__AIN1"
+	(label "D12__AIN1"
 		(at 243.84 33.02 270)
 		(effects
@@
 		)
 	)
-	(label "D12__AIN0"
+	(label "D11__AIN0"
 		(at 246.38 33.02 270)
 		(effects
@@
 		)
 	)
-	(label "D11__AIN4"
+	(label "D10__AIN4"
 		(at 236.22 33.02 270)
 		(effects

Commit message: Another swap.
Connections:
- net A0__AIN2 renamed A0__AIN4
- net A0__AIN4: now also J2.6 (Pin_6); no longer J2.4 (Pin_4)
- net D10__AIN4 renamed D10__AIN2
- net D10__AIN2: now also J2.4 (Pin_4); no longer J2.6 (Pin_6)
Changed lines of the file:
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@@
 		)
 	)
-	(label "A0__AIN2"
+	(label "A0__AIN4"
 		(at 142.24 58.42 180)
 		(effects
@@
 		)
 	)
-	(label "D10__AIN4"
+	(label "D10__AIN2"
 		(at 91.44 68.58 0)
 		(effects
@@
 		)
 	)
-	(label "A0__AIN2"
-		(at 241.3 33.02 270)
+	(label "A0__AIN4"
+		(at 236.22 33.02 270)
 		(effects
 			(font
@@
 		)
 	)
-	(label "D10__AIN4"
-		(at 236.22 33.02 270)
-		(effects
-			(font
+	(label "D10__AIN2"
+		(at 241.3 33.02 270)
+		(effects
+			(font
