File: HW/Ard_Nano_2_LPRS1_MAX1000_Shield/Ard_Nano_2_LPRS1_MAX1000_Shield.kicad_sch (KiCad schematic)
At the start: 3 parts, among them J1 1x14 2.54mm female, J2 1x14 2.54mm female

Commit message: v0.3
Connections:
- net +5V: now also J1.12 (Pin_12)
- net +3V3: no longer names the net of A1.17 (3V3)
- net +3V3: no longer J1.12 (Pin_12)
- net A0__AIN4 renamed A0__AIN2
- net A0__AIN2: now also J2.4 (Pin_4); no longer J2.6 (Pin_6)
- net D10__AIN2 renamed D10__AIN0
- net D10__AIN0: now also J2.2 (Pin_2); no longer J2.4 (Pin_4)
- net D11__AIN0 renamed D11__AIN4
- net D11__AIN4: now also J2.6 (Pin_6); no longer J2.2 (Pin_2)
- net D12__AIN1: no longer names the net of J2.3 (Pin_3)
- net D12__AIN1: no longer A1.15 (D12)
- net D13__AIN3: no longer names the net of A1.16 (D13)
- net D13__AIN3: no longer J2.5 (Pin_5)
- new net D12__AIN3: A1.15 (D12), J2.5 (Pin_5)
- no-connect marks 13 -> 16
Changed lines of the file:
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@@
+	)
+	(no_connect
+		(at 119.38 33.02)
 	)
 	(no_connect
@@
 	)
 	(no_connect
+		(at 104.14 76.2)
+	)
+	(no_connect
+		(at 243.84 45.72)
+	)
+	(no_connect
 		(at 129.54 53.34)
 	)
@@
 	(wire
 		(pts
-			(xy 119.38 26.67) (xy 119.38 33.02)
-		)
-		(stroke
-			(width 0)
-			(type default)
-		)
-	)
-	(wire
-		(pts
 			(xy 91.44 66.04) (xy 104.14 66.04)
 		)
@@
 	(wire
 		(pts
-			(xy 243.84 33.02) (xy 243.84 45.72)
-		)
-		(stroke
-			(width 0)
-			(type default)
-		)
-	)
-	(wire
-		(pts
 			(xy 142.24 68.58) (xy 129.54 68.58)
 		)
@@
 		(pts
 			(xy 223.52 33.02) (xy 223.52 45.72)
-		)
-		(stroke
-			(width 0)
-			(type default)
-		)
-	)
-	(wire
-		(pts
-			(xy 91.44 76.2) (xy 104.14 76.2)
 		)
 		(stroke
@@
 		)
 	)
-	(label "D13__AIN3"
-		(at 238.76 33.02 270)
-		(effects
-			(font
-				(size 1.27 1.27)
-			)
-			(justify right bottom)
-		)
-	)
 	(label "D14"
 		(at 236.22 104.14 90)
@@
 		)
 	)
-	(label "A0__AIN4"
+	(label "A0__AIN2"
 		(at 142.24 58.42 180)
 		(effects
@@
 		)
 	)
-	(label "D13__AIN3"
-		(at 91.44 76.2 0)
-		(effects
-			(font
-				(size 1.27 1.27)
-			)
-			(justify left bottom)
-		)
-	)
-	(label "D11__AIN0"
+	(label "D11__AIN4"
 		(at 91.44 71.12 0)
 		(effects
@@
 		)
 	)
-	(label "D10__AIN2"
+	(label "D10__AIN0"
 		(at 91.44 68.58 0)
 		(effects
@@
 		)
 	)
-	(label "D12__AIN1"
-		(at 91.44 73.66 0)
-		(effects
-			(font
-				(size 1.27 1.27)
-			)
-			(justify left bottom)
-		)
-	)
 	(label "D1"
 		(at 227.33 66.04 90)
@@
 		)
 	)
-	(label "A0__AIN4"
+	(label "D11__AIN4"
 		(at 236.22 33.02 270)
 		(effects
@@
 		)
 	)
-	(label "D12__AIN1"
-		(at 243.84 33.02 270)
+	(label "D12__AIN3"
+		(at 238.76 33.02 270)
 		(effects
 			(font
@@
 		)
 	)
-	(label "D11__AIN0"
+	(label "D10__AIN0"
 		(at 246.38 33.02 270)
 		(effects
@@
 			)
 			(justify right bottom)
+		)
+	)
+	(label "D12__AIN3"
+		(at 91.44 73.66 0)
+		(effects
+			(font
+				(size 1.27 1.27)
+			)
+			(justify left bottom)
 		)
 	)
@@
 		)
 	)
-	(label "D10__AIN2"
+	(label "A0__AIN2"
 		(at 241.3 33.02 270)
 		(effects
@@
 			)
 			(justify left bottom)
-		)
-	)
-	(symbol
-		(lib_id "LPRS1_MAX1000_Shield-rescue:+3V3-power")
-		(at 243.84 125.73 180)
-		(unit 1)
-		(exclude_from_sim no)
-		(in_bom yes)
-		(on_board yes)
-		(dnp no)
-		(property "Reference" "#PWR5"
-			(at 243.84 121.92 0)
-			(effects
-				(font
-					(size 1.27 1.27)
-				)
-				(hide yes)
-			)
-		)
-		(property "Value" "+3V3"
-			(at 243.459 130.1242 0)
-			(effects
-				(font
-					(size 1.27 1.27)
-				)
-			)
-		)
-		(property "Footprint" ""
-			(at 243.84 125.73 0)
-			(effects
-				(font
-					(size 1.27 1.27)
-				)
-				(hide yes)
-			)
-		)
-		(property "Datasheet" ""
-			(at 243.84 125.73 0)
-			(effects
-				(font
-					(size 1.27 1.27)
-				)
-				(hide yes)
-			)
-		)
-		(property "Description" ""
-			(at 243.84 125.73 0)
-			(effects
-				(font
-					(size 1.27 1.27)
-				)
-				(hide yes)
-			)
-		)
-		(pin "1"
-		)
-		(instances
-			(project "Ard_Nano_2_LPRS1_MAX1000_Shield"
-				(path "/f032f0f5-bc12-4ceb-9247-9ea9649022af"
-					(reference "#PWR5")
-					(unit 1)
-				)
-			)
 		)
 	)
@@
 	)
 	(symbol
-		(lib_id "LPRS1_MAX1000_Shield-rescue:+3V3-power")
-		(at 119.38 26.67 0)
+		(lib_id "LPRS1_MAX1000_Shield-rescue:+5V-power")
+		(at 243.84 125.73 180)
 		(unit 1)
 		(exclude_from_sim no)
@@
 		(on_board yes)
 		(dnp no)
-		(property "Reference" "#PWR6"
-			(at 119.38 30.48 0)
-			(effects
-				(font
-					(size 1.27 1.27)
-				)
-				(hide yes)
-			)
-		)
-		(property "Value" "+3V3"
-			(at 119.761 22.2758 0)
+		(property "Reference" "#PWR5"
+			(at 243.84 121.92 0)
+			(effects
+				(font
+					(size 1.27 1.27)
+				)
+				(hide yes)
+			)
+		)
+		(property "Value" "+5V"
+			(at 243.459 130.1242 0)
 			(effects
 				(font
@@
 		)
 		(property "Footprint" ""
-			(at 119.38 26.67 0)
+			(at 243.84 125.73 0)
 			(effects
 				(font
@@
 		)
 		(property "Datasheet" ""
-			(at 119.38 26.67 0)
+			(at 243.84 125.73 0)
 			(effects
 				(font
@@
 		)
 		(property "Description" ""
-			(at 119.38 26.67 0)
+			(at 243.84 125.73 0)
 			(effects
 				(font
@@
 			(project "Ard_Nano_2_LPRS1_MAX1000_Shield"
 				(path "/f032f0f5-bc12-4ceb-9247-9ea9649022af"
-					(reference "#PWR6")
+					(reference "#PWR5")
 					(unit 1)
 				)
