File: HW/LED_Bar_PM_Stepper_Shield/Bank.kicad_sch (KiCad schematic)
At the start: 7 parts, among them J1 JST XH 5pin male socket, J3 JST XH 5pin male socket, U1 ULN2803A

Commit message: Done PCB.
Parts:
- removed C1, C2: 100n, Capacitor_THT:C_Disc_D3.8mm_W2.6mm_P2.50mm, symbol Device:C
- J2: renamed from J1; Comment (none) -> channel 1
- J3: Comment (none) -> channel 0
Connections:
- net +5V: now also D2.12, D2.9
- net GND: now also D2.10, D2.11
- net O1: now also D2.7, J3.3 (Pin_3), U1.12 (O7); no longer D2.1, J3.2 (Pin_2), U1.18 (O1)
- net O2: now also D2.6, J3.4 (Pin_4), U1.13 (O6); no longer D2.2, J3.3 (Pin_3), U1.17 (O2)
- net O3: now also D2.5, J3.5 (Pin_5), U1.14 (O5); no longer D2.3, J3.4 (Pin_4), U1.16 (O3)
- net O4: now also J2.5 (Pin_5); no longer J3.5 (Pin_5)
- net O5: now also D2.3, J2.4 (Pin_4), U1.16 (O3); no longer D2.5, J2.2 (Pin_2), U1.14 (O5)
- net O6: now also D2.2, U1.17 (O2); no longer D2.6, U1.13 (O6)
- net O7: now also D2.1, J2.2 (Pin_2), U1.18 (O1); no longer D2.7, J2.4 (Pin_4), U1.12 (O7)
- net at D2.13: now also RN1.2 (R1); no longer RN1.9 (R8)
- net at D2.14: now also RN1.3 (R2); no longer RN1.8 (R7)
- net at D2.15: now also RN1.4 (R3); no longer RN1.7 (R6)
- net at D2.16: now also RN1.5 (R4); no longer RN1.6 (R5)
- net at D2.17: now also RN1.6 (R5); no longer RN1.5 (R4)
- net at D2.18: now also RN1.7 (R6); no longer RN1.4 (R3)
- net at D2.19: now also RN1.8 (R7); no longer RN1.3 (R2)
- net at D2.20: now also RN1.9 (R8); no longer RN1.2 (R1)
- net B7: now reaches U1.1 (I1)
- net B6: now reaches U1.2 (I2)
- net B5: now reaches U1.3 (I3)
- net B4: now reaches U1.4 (I4)
- net B3: now reaches U1.5 (I5)
- net B2: now reaches U1.6 (I6)
- net B1: now reaches U1.7 (I7)
- net B0: now reaches U1.8 (I8)
- net O8 renamed O0
- net O0: now also J3.2 (Pin_2); no longer J2.5 (Pin_5)
Other:
- moved on the sheet: D2, RN1

Commit message: Correcting PCB
Parts:
- U1: footprint Package_DIP:DIP-20_W7.62mm_Socket -> Package_DIP:DIP-18_W7.62mm_Socket
Changed lines of the file:
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@@
 			)
 		)
-		(property "Footprint" "Package_DIP:DIP-20_W7.62mm_Socket"
+		(property "Footprint" "Package_DIP:DIP-18_W7.62mm_Socket"
 			(at 87.63 77.47 0)
 			(effects

Commit message: PCB corrected.
Parts:
- renumbered D2 to D1, J3 to J1
Connections:
- net GND: no longer D1.10, D1.11
- no-connect marks 0 -> 2
Changed lines of the file:
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@@
 	(generator_version "8.0")
 	(paper "A4")
+	(no_connect
+		(at 124.46 78.74)
+	)
+	(no_connect
+		(at 111.76 78.74)
+	)
 	(wire
 		(pts
@@
 	(wire
 		(pts
-			(xy 109.22 78.74) (xy 111.76 78.74)
-		)
-		(stroke
-			(width 0)
-			(type default)
-		)
-	)
-	(wire
-		(pts
 			(xy 96.52 48.26) (xy 96.52 53.34)
 		)
@@
 		(pts
 			(xy 111.76 58.42) (xy 96.52 58.42)
-		)
-		(stroke
-			(width 0)
-			(type default)
-		)
-	)
-	(wire
-		(pts
-			(xy 127 78.74) (xy 124.46 78.74)
 		)
 		(stroke
@@
 		(on_board yes)
 		(dnp no)
-		(property "Reference" "J3"
+		(property "Reference" "J1"
 			(at 152.4 110.4899 0)
 			(effects
@@
 		(dnp no)
 		(fields_autoplaced yes)
-		(property "Reference" "D2"
+		(property "Reference" "D1"
 			(at 118.11 48.26 0)
 			(effects
@@
 	)
 	(symbol
-		(lib_id "power:GND")
-		(at 109.22 78.74 270)
-		(unit 1)
-		(exclude_from_sim no)
-		(in_bom yes)
-		(on_board yes)
-		(dnp no)
-		(fields_autoplaced yes)
-		(property "Reference" "#PWR9"
-			(at 102.87 78.74 0)
-			(effects
-				(font
-					(size 1.27 1.27)
-				)
-				(hide yes)
-			)
-		)
-		(property "Value" "GND"
-			(at 105.41 78.7399 90)
-			(effects
-				(font
-					(size 1.27 1.27)
-				)
-				(justify right)
-			)
-		)
-		(property "Footprint" ""
-			(at 109.22 78.74 0)
-			(effects
-				(font
-					(size 1.27 1.27)
-				)
-				(hide yes)
-			)
-		)
-		(property "Datasheet" ""
-			(at 109.22 78.74 0)
-			(effects
-				(font
-					(size 1.27 1.27)
-				)
-				(hide yes)
-			)
-		)
-		(property "Description" "Power symbol creates a global label with name \"GND\" , ground"
-			(at 109.22 78.74 0)
-			(effects
-				(font
-					(size 1.27 1.27)
-				)
-				(hide yes)
-			)
-		)
-		(pin "1"
-		)
-		(instances
-			(project ""
-				(path "/f032f0f5-bc12-4ceb-9247-9ea9649022af/bf5551d3-91c4-4f6c-b676-3570ac7e1d00"
-					(reference "#PWR9")
-					(unit 1)
-				)
-				(path "/f032f0f5-bc12-4ceb-9247-9ea9649022af/f6cb011b-05f3-41a8-901e-17013340861f"
-					(reference "#PWR10")
-					(unit 1)
-				)
-			)
-		)
-	)
-	(symbol
 		(lib_id "power:+5V")
 		(at 109.22 76.2 90)
@@
 					(unit 1)
 				)
-			)
-		)
-	)
-	(symbol
-		(lib_id "power:GND")
-		(at 127 78.74 90)
-		(unit 1)
-		(exclude_from_sim no)
-		(in_bom yes)
-		(on_board yes)
-		(dnp no)
-		(fields_autoplaced yes)
-		(property "Reference" "#PWR11"
-			(at 133.35 78.74 0)
-			(effects
-				(font
-					(size 1.27 1.27)
-				)
-				(hide yes)
-			)
-		)
-		(property "Value" "GND"
-			(at 130.81 78.7401 90)
-			(effects
-				(font
-					(size 1.27 1.27)
-				)
-				(justify right)
-			)
-		)
-		(property "Footprint" ""
-			(at 127 78.74 0)
-			(effects
-				(font
-					(size 1.27 1.27)
-				)
-				(hide yes)
-			)
-		)
-		(property "Datasheet" ""
-			(at 127 78.74 0)
-			(effects
-				(font
-					(size 1.27 1.27)
-				)
-				(hide yes)
-			)
-		)
-		(property "Description" "Power symbol creates a global label with name \"GND\" , ground"
-			(at 127 78.74 0)
-			(effects
-				(font
-					(size 1.27 1.27)
-				)
-				(hide yes)
-			)
-		)
-		(pin "1"
-		)
-		(instances
-			(project "LED_Bar_PM_Stepper_Shield"
-				(path "/f032f0f5-bc12-4ceb-9247-9ea9649022af/bf5551d3-91c4-4f6c-b676-3570ac7e1d00"
-					(reference "#PWR11")
-					(unit 1)
-				)
-				(path "/f032f0f5-bc12-4ceb-9247-9ea9649022af/f6cb011b-05f3-41a8-901e-17013340861f"
-					(reference "#PWR12")
-					(unit 1)
-				)

Commit message: Connector orientations correction.
Connections:
- net +5V: now also J1.5 (Pin_5), J2.5 (Pin_5); no longer J1.1 (Pin_1), J2.1 (Pin_1)
- net O0: now also J1.4 (Pin_4); no longer J1.2 (Pin_2)
- net O2: now also J1.2 (Pin_2); no longer J1.4 (Pin_4)
- net O3: now also J1.1 (Pin_1); no longer J1.5 (Pin_5)
- net O4: now also J2.1 (Pin_1); no longer J2.5 (Pin_5)
- net O5: now also J2.2 (Pin_2); no longer J2.4 (Pin_4)
- net O7: now also J2.4 (Pin_4); no longer J2.2 (Pin_2)
Changed lines of the file:
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@@
 		(lib_id "Connector_Generic:Conn_01x05")
 		(at 149.86 142.24 0)
+		(mirror x)
 		(unit 1)
 		(exclude_from_sim no)
@@
 		(dnp no)
 		(property "Reference" "J2"
-			(at 152.4 140.9699 0)
+			(at 152.4 143.5101 0)
 			(effects
 				(font
@@
 		)
 		(property "Value" "JST XH 5pin male socket"
-			(at 152.4 143.5099 0)
+			(at 152.4 140.9701 0)
 			(effects
 				(font
@@
 		)
 		(property "Comment" "channel 1"
-			(at 159.004 146.558 0)
+			(at 159.004 137.922 0)
 			(effects
 				(font
@@
 		(lib_id "Connector_Generic:Conn_01x05")
 		(at 149.86 111.76 0)
+		(mirror x)
 		(unit 1)
 		(exclude_from_sim no)
@@
 		(dnp no)
 		(property "Reference" "J1"
-			(at 152.4 110.4899 0)
+			(at 152.4 113.0301 0)
 			(effects
 				(font
@@
 		)
 		(property "Value" "JST XH 5pin male socket"
-			(at 152.4 113.0299 0)
+			(at 152.4 110.4901 0)
 			(effects
 				(font
@@
 		)
 		(property "Comment" "channel 0"
-			(at 160.782 116.586 0)
-			(effects
-				(font
+			(at 160.782 106.934 0)
+			(effects
+				(font
